File: yellow_fuzz_dev/yellow_fuzz_dev.sch (KiCad schematic (older format))
At the start: 150 parts

Commit message: reviewing all filter setpoints, just made it to distortion section
Parts:
- removed C?: 15n, Capacitor_SMD:C_0603_1608Metric_Pad1.05x0.95mm_HandSolder, symbol Device:C
- removed C?: 220p, Capacitor_SMD:C_0603_1608Metric_Pad1.05x0.95mm_HandSolder, symbol Device:C
- added C?: 1.0u, Capacitor_SMD:C_0603_1608Metric_Pad1.05x0.95mm_HandSolder, symbol Device:C
- added C?: 100p, Capacitor_SMD:C_0603_1608Metric_Pad1.05x0.95mm_HandSolder, symbol Device:C
Connections:
- net at Q?.2 (D), R?.2: now also C?.2
- net at R?.2, U?.3: now also C?.1
- net at R?.1, R?.2, U?.1: now also C?.1
- net at C?.1, R?.2, U?.2: now also C?.2
Changed lines of the file:
@@
-$EndComp
-$Comp
-L Device:C C?
-U 1 1 5E3D7DDB
-P 7850 3800
-F 0 "C?" H 7965 3937 50  0000 L CNN
-F 1 "220p" H 7950 3850 50  0000 L CNN
-F 2 "Capacitor_SMD:C_0603_1608Metric_Pad1.05x0.95mm_HandSolder" H 7888 3650 50  0001 C CNN
-F 3 "~" H 7850 3800 50  0001 C CNN
-F 4 "Yageo" H 7850 3800 50  0001 C CNN "Manufacturer"
-F 5 "CC0603KRX7R9BB221" H 7850 3800 50  0001 C CNN "Manufacturer PN"
-F 6 "Digi-Key" H 7850 3800 50  0001 C CNN "Supplier"
-F 7 "311-1077-1-ND" H 7850 3800 50  0001 C CNN "Supplier PN"
-F 8 "0603" H 7965 3755 50  0000 L CNN "Package"
-F 9 "50V" H 7965 3664 50  0000 L CNN "Voltage"
-	1    7850 3800
-	0    1    1    0
 $EndComp
 $Comp
@@
 	1    6650 6700
 	1    0    0    -1
-$EndComp
-$Comp
-L Device:C C?
-U 1 1 5E3CC437
-P 6400 7000
-F 0 "C?" H 6515 7137 50  0000 L CNN
-F 1 "15n" H 6500 7050 50  0000 L CNN
-F 2 "Capacitor_SMD:C_0603_1608Metric_Pad1.05x0.95mm_HandSolder" H 6438 6850 50  0001 C CNN
-F 3 "~" H 6400 7000 50  0001 C CNN
-F 4 "Yageo" H 6400 7000 50  0001 C CNN "Manufacturer"
-F 5 "CC0603KRX7R9BB153" H 6400 7000 50  0001 C CNN "Manufacturer PN"
-F 6 "Digi-Key" H 6400 7000 50  0001 C CNN "Supplier"
-F 7 "311-1430-1-ND" H 6400 7000 50  0001 C CNN "Supplier PN"
-F 8 "0603" H 6515 6955 50  0000 L CNN "Package"
-F 9 "50V" H 6515 6864 50  0000 L CNN "Voltage"
-	1    6400 7000
-	0    1    1    0
 $EndComp
 $Comp
@@
 Wire Wire Line
 	16200 10650 16200 10750
+$Comp
+L Device:C C?
+U 1 1 60FEC222
+P 6400 7000
+F 0 "C?" H 6515 7137 50  0000 L CNN
+F 1 "1.0u" H 6500 7050 50  0000 L CNN
+F 2 "Capacitor_SMD:C_0603_1608Metric_Pad1.05x0.95mm_HandSolder" H 6438 6850 50  0001 C CNN
+F 3 "~" H 6400 7000 50  0001 C CNN
+F 4 "Yageo" H 6400 7000 50  0001 C CNN "Manufacturer"
+F 5 "CC0603ZRY5V7BB105" H 6400 7000 50  0001 C CNN "Manufacturer PN"
+F 6 "Digi-Key" H 6400 7000 50  0001 C CNN "Supplier"
+F 7 "311-1372-1-ND" H 6400 7000 50  0001 C CNN "Supplier PN"
+F 8 "0603" H 6515 6955 50  0000 L CNN "Package"
+F 9 "16V" H 6515 6864 50  0000 L CNN "Voltage"
+	1    6400 7000
+	0    1    1    0
+$EndComp
+$Comp
+L Device:C C?
+U 1 1 60FECBAA
+P 7850 3800
+F 0 "C?" H 7965 3937 50  0000 L CNN
+F 1 "100p" H 7950 3850 50  0000 L CNN
+F 2 "Capacitor_SMD:C_0603_1608Metric_Pad1.05x0.95mm_HandSolder" H 7888 3650 50  0001 C CNN
+F 3 "~" H 7850 3800 50  0001 C CNN
+F 4 "Yageo" H 7850 3800 50  0001 C CNN "Manufacturer"
+F 5 "CC0603JRNPO9BN101" H 7850 3800 50  0001 C CNN "Manufacturer PN"
+F 6 "Digi-Key" H 7850 3800 50  0001 C CNN "Supplier"
+F 7 "311-1069-1-ND" H 7850 3800 50  0001 C CNN "Supplier PN"
+F 8 "0603" H 7965 3755 50  0000 L CNN "Package"
+F 9 "50V" H 7965 3664 50  0000 L CNN "Voltage"
+	1    7850 3800
+	0    1    1    0
+$EndComp
 $EndSCHEMATC
