File: yellow_fuzz_dev/yellow_fuzz_dev.sch (KiCad schematic (older format))
At the start: 133 parts, among them J1 PJ-202A, J2 RA49B11, J3 SN49B12B, P1 3386P-1-204TLF, P2 PTV112-4420A-A104, P3 3362P-1-102TLF, P4 3362P-1-102TLF, Q1 DMN2041L, Q10 BC817-25-TP, Q11 NSVJ3910SB3T1GOSCT-ND, Q12 BC817-25-TP, Q13 BC817-25-TP, Q14 NSVJ3910SB3T1GOSCT-ND, Q2 NSVJ3910SB3T1GOSCT-ND, Q3 DMN2041L, Q4 NSVJ3910SB3T1GOSCT-ND, Q5 BC817-25-TP, Q6 BC817-25-TP, Q7 BC817-25-TP, Q8 BC817-25-TP, Q9 BC817-25-TP, SW1 SW_SP3T_A24JP, SW2 SW_SP3T_A24JP, SW3 SW_SP3T_A24JP, SW4 SW_SPST_A11JP, SW5 SW_SPST_A11JP, U1 TL072CP, U2 TL072CP

Commit message: corrected BOM fields and generated BOM
Parts:
- BAT1: Digi-Key_PN BC9VPC-ND -> (none); MPN BC9VPC -> (none); Manufacturer PN (none) -> BC9VPC; Supplier (none) -> Digi-Key; Supplier PN (none) -> BC9VPC-ND
- D1, D10, D11: Manufacturer PN (none) -> BAS16WT1G; Manufacturer Part Number BAS16WT1G -> (none); Supplier PN (none) -> BAS16WT1GOSCT-ND; Supplier Part Number BAS16WT1GOSCT-ND -> (none)
- D2: Manufacturer (none) -> Panasonic Electronic Components; Manufacturer PN (none) -> DZ2S056M0L; Supplier (none) -> Digi-Key; Supplier PN (none) -> DZ2S056M0LCT-ND
- D3, D6, D9: Digi-Key_PN 754-1489-ND -> (none); MPN WP7113QBC/D -> (none); Manufacturer PN (none) -> WP7113QBC/D; Supplier (none) -> Digi-Key; Supplier PN (none) -> 754-1489-ND
- D4, D7: Digi-Key_PN 1N4148FS-ND -> (none); MPN 1N4148 -> (none); Manufacturer PN (none) -> 1N4148; Supplier (none) -> Digi-Key; Supplier PN (none) -> 1N4148FS-ND
- D5, D8: Digi-Key_PN 2368-1N34A-ND -> (none); MPN 1N34A -> (none); Manufacturer PN (none) -> 1N34A; Supplier (none) -> Digi-Key; Supplier PN (none) -> 2368-1N34A-ND
- J1: Digi-Key_PN CP-202A-ND -> (none); MPN PJ-202A -> (none); Manufacturer PN (none) -> PJ-202A; Supplier (none) -> Digi-Key; Supplier PN (none) -> CP-202A-ND
- J2: Manufacturer (none) -> Switchcraft; Manufacturer PN (none) -> RA49B11; Supplier (none) -> Digi-Key; Supplier PN (none) -> SC2546-ND
- J3: Digi-Key_PN SC1522-ND -> (none); MPN SN49B12B -> (none); Manufacturer PN (none) -> SN49B12B; Supplier (none) -> Digi-Key; Supplier PN (none) -> SC1522-ND
- P1: Digi-Key_PN 3386P-1-204TLF-ND -> (none); MPN 3386P-1-204TLF -> (none); Manufacturer PN (none) -> 3386P-1-204TLF; Supplier (none) -> Digi-Key; Supplier PN (none) -> 3386P-1-204TLF-ND
- P3, P4: Digi-Key_PN 3362P-1-102TLF-ND -> (none); MPN 3362P-1-102TLF -> (none); Manufacturer PN (none) -> 3362P-1-102TLF; Supplier (none) -> Digi-Key; Supplier PN (none) -> 3362P-1-102TLF-ND
- Q1, Q3: Manufacturer (none) -> Diodes Incorporated; Manufacturer PN (none) -> DMN2041L-7; Supplier (none) -> Digi-Key; Supplier PN (none) -> DMN2041L-7DICT-ND
- Q10, Q12, Q13, Q5, Q6, Q7, Q8, Q9: Digi-Key_PN BC817-25-TPMSCT-ND -> (none); MPN BC817-25-TP -> (none); Manufacturer PN (none) -> BC817-25-TP; Supplier (none) -> Digi-Key; Supplier PN (none) -> BC817-25-TPMSCT-ND
- Q11, Q14, Q2, Q4: Digi-Key_PN J113FS-ND -> (none); MPN NSVJ3910SB3T1G -> (none); Manufacturer PN (none) -> NSVJ3910SB3T1G; Supplier (none) -> Digi-Key; Supplier PN (none) -> J113FS-ND
- S1: Digi-Key_PN 450-1650-ND -> (none); MPN 1825910-6 -> (none); Manufacturer PN (none) -> 1825910-6; Supplier (none) -> Digi-Key; Supplier PN (none) -> 450-1650-ND
- SW1, SW2, SW3: Manufacturer PN (none) -> A24JP; Manufacturer Part Number A24JP -> (none); Supplier PN (none) -> 360-3408-ND; Supplier Part Number 360-3408-ND -> (none)
- SW4, SW5: Manufactuer PN (none) -> A11JP; Manufactuer Part Number A11JP -> (none); Supplier PN (none) -> 360-2973-ND; Supplier Part Number 360-2973-ND -> (none)
- U1, U2: Digi-Key_PN 296-1775-5-ND -> (none); MPN TL072CP -> (none); Manufacturer PN (none) -> TL072CP; Supplier (none) -> Digi-Key; Supplier PN (none) -> 296-1775-5-ND
