File: yellow_fuzz_dev/tone_block.sch (KiCad schematic (older format))
At the start: 31 parts, among them P5 PTV111-4420A-A104, P6 PTV111-4420A-A104, P7 PTV111-4420A-A104, P8 PTV112-4420A-A503, P9 PTV111-4420A-A503, U3 TL072CP, U4 TL072CP

Commit message: corrected BOM fields and generated BOM
Parts:
- P5, P6, P7: Manufacturer PN (none) -> PTV111-4420A-A104; Manufacturer Part Number PTV111-4420A-A104 -> (none); Supplier PN (none) -> 652-PTV111-4420AA104; Supplier Part Number 652-PTV111-4420AA104 -> (none)
- P8: Manufacturer PN (none) -> PTV112-4420A-A503; Manufacturer Part Number PTV112-4420A-A503 -> (none); Supplier PN (none) -> 652-PTV112-4420AA503; Supplier Part Number 652-PTV112-4420AA503 -> (none)
- P9: Manufacturer PN (none) -> PTV111-4420A-A503; Manufacturer Part Number PTV111-4420A-A503 -> (none); Supplier PN (none) -> 652-PTV111-4420AA503; Supplier Part Number 652-PTV111-4420AA503 -> (none)
- U3, U4: Digi-Key_PN 296-1775-5-ND -> (none); MPN TL072CP -> (none); Manufacturer PN (none) -> TL072CP; Supplier (none) -> Digi-Key; Supplier PN (none) -> 296-1775-5-ND
Changed lines of the file:
@@
 F 2 "yellow_fuzz_dev:DIP-8_W7.62mm" H 6450 4650 60  0001 L CNN
 F 3 "http://www.ti.com/general/docs/suppproductinfo.tsp?distId=10&gotoUrl=http%3A%2F%2Fwww.ti.com%2Flit%2Fgpn%2Ftl071a" H 6450 4750 60  0001 L CNN
-F 4 "296-1775-5-ND" H 6450 4850 60  0001 L CNN "Digi-Key_PN"
-F 5 "TL072CP" H 6450 4950 60  0001 L CNN "MPN"
+F 4 "296-1775-5-ND" H 6450 4850 60  0001 L CNN "Supplier PN"
+F 5 "TL072CP" H 6450 4950 60  0001 L CNN "Manufacturer PN"
 F 6 "Integrated Circuits (ICs)" H 6450 5050 60  0001 L CNN "Category"
 F 7 "Linear - Amplifiers - Instrumentation, OP Amps, Buffer Amps" H 6450 5150 60  0001 L CNN "Family"
@@
 F 11 "Texas Instruments" H 6450 5550 60  0001 L CNN "Manufacturer"
 F 12 "Active" H 6450 5650 60  0001 L CNN "Status"
+F 13 "Digi-Key" H 6250 4450 50  0001 C CNN "Supplier"
 	1    6250 4450
 	1    0    0    -1
@@
 F 2 "yellow_fuzz_dev:DIP-8_W7.62mm" H 3550 6850 60  0001 L CNN
 F 3 "http://www.ti.com/general/docs/suppproductinfo.tsp?distId=10&gotoUrl=http%3A%2F%2Fwww.ti.com%2Flit%2Fgpn%2Ftl071a" H 3550 6950 60  0001 L CNN
-F 4 "296-1775-5-ND" H 3550 7050 60  0001 L CNN "Digi-Key_PN"
-F 5 "TL072CP" H 3550 7150 60  0001 L CNN "MPN"
+F 4 "296-1775-5-ND" H 3550 7050 60  0001 L CNN "Supplier PN"
+F 5 "TL072CP" H 3550 7150 60  0001 L CNN "Manufacturer PN"
 F 6 "Integrated Circuits (ICs)" H 3550 7250 60  0001 L CNN "Category"
 F 7 "Linear - Amplifiers - Instrumentation, OP Amps, Buffer Amps" H 3550 7350 60  0001 L CNN "Family"
@@
 F 11 "Texas Instruments" H 3550 7750 60  0001 L CNN "Manufacturer"
 F 12 "Active" H 3550 7850 60  0001 L CNN "Status"
+F 13 "Digi-Key" V 3350 6650 50  0001 C CNN "Supplier"
 	2    3350 6650
 	0    1    1    0
@@
 F 2 "yellow_fuzz_dev:DIP-8_W7.62mm" H 12300 5450 60  0001 L CNN
 F 3 "http://www.ti.com/general/docs/suppproductinfo.tsp?distId=10&gotoUrl=http%3A%2F%2Fwww.ti.com%2Flit%2Fgpn%2Ftl071a" H 12300 5550 60  0001 L CNN
-F 4 "296-1775-5-ND" H 12300 5650 60  0001 L CNN "Digi-Key_PN"
-F 5 "TL072CP" H 12300 5750 60  0001 L CNN "MPN"
+F 4 "296-1775-5-ND" H 12300 5650 60  0001 L CNN "Supplier PN"
+F 5 "TL072CP" H 12300 5750 60  0001 L CNN "Manufacturer PN"
 F 6 "Integrated Circuits (ICs)" H 12300 5850 60  0001 L CNN "Category"
 F 7 "Linear - Amplifiers - Instrumentation, OP Amps, Buffer Amps" H 12300 5950 60  0001 L CNN "Family"
@@
 F 11 "Texas Instruments" H 12300 6350 60  0001 L CNN "Manufacturer"
 F 12 "Active" H 12300 6450 60  0001 L CNN "Status"
+F 13 "Digi-Key" H 12100 5250 50  0001 C CNN "Supplier"
 	2    12100 5250
 	-1   0    0    -1
@@
 F 2 "yellow_fuzz_dev:DIP-8_W7.62mm" H 8650 4750 60  0001 L CNN
 F 3 "http://www.ti.com/general/docs/suppproductinfo.tsp?distId=10&gotoUrl=http%3A%2F%2Fwww.ti.com%2Flit%2Fgpn%2Ftl071a" H 8650 4850 60  0001 L CNN
-F 4 "296-1775-5-ND" H 8650 4950 60  0001 L CNN "Digi-Key_PN"
-F 5 "TL072CP" H 8650 5050 60  0001 L CNN "MPN"
+F 4 "296-1775-5-ND" H 8650 4950 60  0001 L CNN "Supplier PN"
+F 5 "TL072CP" H 8650 5050 60  0001 L CNN "Manufacturer PN"
 F 6 "Integrated Circuits (ICs)" H 8650 5150 60  0001 L CNN "Category"
 F 7 "Linear - Amplifiers - Instrumentation, OP Amps, Buffer Amps" H 8650 5250 60  0001 L CNN "Family"
@@
 F 11 "Texas Instruments" H 8650 5650 60  0001 L CNN "Manufacturer"
 F 12 "Active" H 8650 5750 60  0001 L CNN "Status"
+F 13 "Digi-Key" H 8450 4550 50  0001 C CNN "Supplier"
 	1    8450 4550
 	1    0    0    -1
@@
 F 3 "https://www.mouser.com/datasheet/2/54/PTVPTT-56034.pdf" H 10450 7050 60  0001 L CNN
 F 4 "Bourns" H 10450 7150 60  0001 L CNN "Manufacturer"
-F 5 "PTV112-4420A-A503" H 10450 7250 60  0001 L CNN "Manufacturer Part Number"
+F 5 "PTV112-4420A-A503" H 10450 7250 60  0001 L CNN "Manufacturer PN"
 F 6 "Mouser" H 10450 7350 60  0001 L CNN "Supplier"
-F 7 "652-PTV112-4420AA503" H 10450 7450 60  0001 L CNN "Supplier Part Number"
+F 7 "652-PTV112-4420AA503" H 10450 7450 60  0001 L CNN "Supplier PN"
 F 8 "Dual" V 10050 6650 50  0000 R CNN "Gangs"
 F 9 "Log" V 10150 6650 50  0000 R CNN "Taper"
@@
 F 3 "https://www.mouser.com/datasheet/2/54/PTVPTT-56034.pdf" H 11150 6350 60  0001 L CNN
 F 4 "Bourns" H 11150 6450 60  0001 L CNN "Manufacturer"
-F 5 "PTV112-4420A-A503" H 11150 6550 60  0001 L CNN "Manufacturer Part Number"
+F 5 "PTV112-4420A-A503" H 11150 6550 60  0001 L CNN "Manufacturer PN"
 F 6 "Mouser" H 11150 6650 60  0001 L CNN "Supplier"
-F 7 "652-PTV112-4420AA503" H 11150 6750 60  0001 L CNN "Supplier Part Number"
+F 7 "652-PTV112-4420AA503" H 11150 6750 60  0001 L CNN "Supplier PN"
 F 8 "Dual" H 10900 5700 50  0000 C CNN "Gangs"
 F 9 "Log" H 10900 5600 50  0000 C CNN "Taper"
@@
 F 3 "https://www.mouser.com/datasheet/2/54/PTVPTT-56034.pdf" H 13150 5500 60  0001 L CNN
 F 4 "Bourns" H 13150 5600 60  0001 L CNN "Manufacturer"
-F 5 "PTV111-4420A-A503" H 13150 5700 60  0001 L CNN "Manufacturer Part Number"
+F 5 "PTV111-4420A-A503" H 13150 5700 60  0001 L CNN "Manufacturer PN"
 F 6 "Mouser" H 13150 5800 60  0001 L CNN "Supplier"
-F 7 "652-PTV111-4420AA503" H 13150 5900 60  0001 L CNN "Supplier Part Number"
+F 7 "652-PTV111-4420AA503" H 13150 5900 60  0001 L CNN "Supplier PN"
 F 8 "Single" H 12350 5450 50  0001 L CNN "Gangs"
 F 9 "Log" V 12693 5012 50  0000 R CNN "Taper"
@@
 F 3 "https://www.mouser.com/datasheet/2/54/PTVPTT-56034.pdf" H 8800 6600 60  0001 L CNN
 F 4 "Bourns" H 8800 6700 60  0001 L CNN "Manufacturer"
-F 5 "PTV111-4420A-A104" H 8800 6800 60  0001 L CNN "Manufacturer Part Number"
+F 5 "PTV111-4420A-A104" H 8800 6800 60  0001 L CNN "Manufacturer PN"
 F 6 "Mouser" H 8800 6900 60  0001 L CNN "Supplier"
-F 7 "652-PTV111-4420AA104" H 8800 7000 60  0001 L CNN "Supplier Part Number"
+F 7 "652-PTV111-4420AA104" H 8800 7000 60  0001 L CNN "Supplier PN"
 F 8 "Single" H 8000 6550 50  0001 L CNN "Gangs"
 F 9 "Log" H 8550 6700 50  0000 C CNN "Taper"
@@
 F 3 "https://www.mouser.com/datasheet/2/54/PTVPTT-56034.pdf" H 5300 3450 60  0001 L CNN
 F 4 "Bourns" H 5300 3550 60  0001 L CNN "Manufacturer"
-F 5 "PTV111-4420A-A104" H 5300 3650 60  0001 L CNN "Manufacturer Part Number"
+F 5 "PTV111-4420A-A104" H 5300 3650 60  0001 L CNN "Manufacturer PN"
 F 6 "Mouser" H 5300 3750 60  0001 L CNN "Supplier"
-F 7 "652-PTV111-4420AA104" H 5300 3850 60  0001 L CNN "Supplier Part Number"
+F 7 "652-PTV111-4420AA104" H 5300 3850 60  0001 L CNN "Supplier PN"
 F 8 "Single" H 4500 3400 50  0001 L CNN "Gangs"
 F 9 "Log" V 4800 2900 50  0000 C CNN "Taper"
@@
 F 3 "https://www.mouser.com/datasheet/2/54/PTVPTT-56034.pdf" H 5300 5550 60  0001 L CNN
 F 4 "Bourns" H 5300 5650 60  0001 L CNN "Manufacturer"
-F 5 "PTV111-4420A-A104" H 5300 5750 60  0001 L CNN "Manufacturer Part Number"
+F 5 "PTV111-4420A-A104" H 5300 5750 60  0001 L CNN "Manufacturer PN"
 F 6 "Mouser" H 5300 5850 60  0001 L CNN "Supplier"
-F 7 "652-PTV111-4420AA104" H 5300 5950 60  0001 L CNN "Supplier Part Number"
+F 7 "652-PTV111-4420AA104" H 5300 5950 60  0001 L CNN "Supplier PN"
 F 8 "Single" H 4500 5500 50  0001 L CNN "Gangs"
 F 9 "Log" V 5000 5000 50  0000 C CNN "Taper"
